File: kicad/nts_player/nts_player.kicad_sch (KiCad schematic)
At the start: 95 parts, among them J1 SJ1-3523N, J2 RCJ-2123, SW1 PEC11R-4120F-S0018, U1 ESP32-S3-DEV-KIT-N16R8, U2 LM66100DCKR, U3 TPS7A2033PDBVR, U4 TPS22918DBVR, U5 SN74AHCT1G125DBVR, U6 PCM5122PWR

Commit message: feat: change usb
Parts:
- removed USB1: USB4105-GF-A-120, lcsc:USB-C-SMD_MC-311D, symbol lcsc:USB4105-GF-A-120
- added USB2: KH-TYPE-C-16P, lcsc:USB-C-SMD_KH-TYPE-C-16P, symbol lcsc:KH-TYPE-C-16P
Connections:
- net GND: now also R12.1, USB2.1 (EP), USB2.2 (EP), USB2.3 (EP), USB2.4 (EP), USB2.A1 (GND), USB2.A12 (GND), USB2.B1 (GND), USB2.B12 (GND); no longer R12.2
- net VBUS: now reaches C6.2, C7.1, D1.1 (K), U2.1 (VIN)
- net VBUS: now also USB2.A4 (VBUS), USB2.A9 (VBUS), USB2.B4 (VBUS), USB2.B9 (VBUS)
- net at R13.1: now also USB2.B5 (CC2)
- new net: R12.2, USB2.A5 (CC1)
- no-connect marks 29 -> 35
Other:
- moved on the sheet: SW1, U2

Commit message: fix: ERC errors
Parts:
- renumbered LED11 to LED10, LED14 to LED11, LED17 to LED12, LED3 to LED13, LED6 to LED14, LED9 to LED15, LED12 to LED16, LED15 to LED17, LED4 to LED2, LED7 to LED3, LED10 to LED4, LED13 to LED5, LED16 to LED6, LED2 to LED7, LED5 to LED8, LED8 to LED9
Connections:
- net +5V_LDO_IN: now reaches C8.1, FB1.2, U3.1 (IN)
- no-connect marks 35 -> 36
Other:
- note added: "DAC + OUTPUTS"
- note added: "DAC POWER"
- note added: "ENCODER"
- note added: "LED ARRAY"
- note added: "LED POWER/DATA"
- note added: "MCU"
- note added: "USB-C POWER"
- moved on the sheet: C20, C24, C27, C31

Commit message: feat: add footprint for esp32
Parts:
- U1: footprint (none) -> waveshare:ESP32-S3-DEV-KIT-NXR8
Connections:
- net GND: now also U1.44 (GND); no longer U1.43 (GND)
- no-connect marks 36 -> 40
Changed lines of the file:
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@@
 	)
 	(no_connect
+		(at 78.74 50.8)
+	)
+	(no_connect
 		(at 242.57 27.94)
 	)
@@
 	)
 	(no_connect
+		(at 31.75 63.5)
+	)
+	(no_connect
+		(at 55.88 34.29)
+	)
+	(no_connect
 		(at 78.74 53.34)
 	)
@@
 	)
 	(no_connect
+		(at 11.43 57.15)
+	)
+	(no_connect
 		(at 78.74 83.82)
 	)
@@
 			)
 		)
-		(property "Footprint" ""
+		(property "Footprint" "waveshare:ESP32-S3-DEV-KIT-NXR8"
 			(at 53.34 43.18 0)
 			(hide yes)
@@
 		(pin "22"
 		)
+		(pin "44"
+		)
 		(instances

Commit message: fix: assign 3d models
Parts:
- LED1, LED10, LED11, LED12, LED13, LED14, LED15, LED16, LED17, LED18, LED2, LED3, LED4, LED5, LED6, LED7, LED8, LED9: footprint lcsc:LED-SMD_4P-L2.2-W2.0-P1.00_WS2815C-2020-4P -> lcsc:WS2815B-2020-V6
Changed lines of the file:
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@@
 			)
 		)
-		(property "Footprint" "lcsc:LED-SMD_4P-L2.2-W2.0-P1.00_WS2815C-2020-4P"
+		(property "Footprint" "lcsc:WS2815B-2020-V6"
 			(at 135.89 78.74 0)
 			(hide yes)
@@
 			)
 		)
-		(property "Footprint" "lcsc:LED-SMD_4P-L2.2-W2.0-P1.00_WS2815C-2020-4P"
+		(property "Footprint" "lcsc:WS2815B-2020-V6"
 			(at 200.66 78.74 0)
 			(hide yes)
@@
 			)
 		)
-		(property "Footprint" "lcsc:LED-SMD_4P-L2.2-W2.0-P1.00_WS2815C-2020-4P"
+		(property "Footprint" "lcsc:WS2815B-2020-V6"
 			(at 135.89 101.6 0)
 			(hide yes)
@@
 			)
 		)
-		(property "Footprint" "lcsc:LED-SMD_4P-L2.2-W2.0-P1.00_WS2815C-2020-4P"
+		(property "Footprint" "lcsc:WS2815B-2020-V6"
 			(at 114.3 78.74 0)
 			(hide yes)
@@
 			)
 		)
-		(property "Footprint" "lcsc:LED-SMD_4P-L2.2-W2.0-P1.00_WS2815C-2020-4P"
+		(property "Footprint" "lcsc:WS2815B-2020-V6"
 			(at 200.66 123.19 0)
 			(hide yes)
@@
 			)
 		)
-		(property "Footprint" "lcsc:LED-SMD_4P-L2.2-W2.0-P1.00_WS2815C-2020-4P"
+		(property "Footprint" "lcsc:WS2815B-2020-V6"
 			(at 114.3 101.6 0)
 			(hide yes)
@@
 			)
 		)
-		(property "Footprint" "lcsc:LED-SMD_4P-L2.2-W2.0-P1.00_WS2815C-2020-4P"
+		(property "Footprint" "lcsc:WS2815B-2020-V6"
 			(at 157.48 123.19 0)
 			(hide yes)
@@
 			)
 		)
-		(property "Footprint" "lcsc:LED-SMD_4P-L2.2-W2.0-P1.00_WS2815C-2020-4P"
+		(property "Footprint" "lcsc:WS2815B-2020-V6"
 			(at 222.25 78.74 0)
 			(hide yes)
@@
 			)
 		)
-		(property "Footprint" "lcsc:LED-SMD_4P-L2.2-W2.0-P1.00_WS2815C-2020-4P"
+		(property "Footprint" "lcsc:WS2815B-2020-V6"
 			(at 114.3 123.19 0)
 			(hide yes)
@@
 			)
 		)
-		(property "Footprint" "lcsc:LED-SMD_4P-L2.2-W2.0-P1.00_WS2815C-2020-4P"
+		(property "Footprint" "lcsc:WS2815B-2020-V6"
 			(at 179.07 78.74 0)
 			(hide yes)
@@
 			)
 		)
-		(property "Footprint" "lcsc:LED-SMD_4P-L2.2-W2.0-P1.00_WS2815C-2020-4P"
+		(property "Footprint" "lcsc:WS2815B-2020-V6"
 			(at 179.07 123.19 0)
 			(hide yes)
@@
 			)
 		)
-		(property "Footprint" "lcsc:LED-SMD_4P-L2.2-W2.0-P1.00_WS2815C-2020-4P"
+		(property "Footprint" "lcsc:WS2815B-2020-V6"
 			(at 157.48 101.6 0)
 			(hide yes)
@@
 			)
 		)
-		(property "Footprint" "lcsc:LED-SMD_4P-L2.2-W2.0-P1.00_WS2815C-2020-4P"
+		(property "Footprint" "lcsc:WS2815B-2020-V6"
 			(at 179.07 101.6 0)
 			(hide yes)
@@
 			)
 		)
-		(property "Footprint" "lcsc:LED-SMD_4P-L2.2-W2.0-P1.00_WS2815C-2020-4P"
+		(property "Footprint" "lcsc:WS2815B-2020-V6"
 			(at 200.66 101.6 0)
 			(hide yes)
@@
 			)
 		)
-		(property "Footprint" "lcsc:LED-SMD_4P-L2.2-W2.0-P1.00_WS2815C-2020-4P"
+		(property "Footprint" "lcsc:WS2815B-2020-V6"
 			(at 222.25 123.19 0)
 			(hide yes)
@@
 			)
 		)
-		(property "Footprint" "lcsc:LED-SMD_4P-L2.2-W2.0-P1.00_WS2815C-2020-4P"
+		(property "Footprint" "lcsc:WS2815B-2020-V6"
 			(at 222.25 101.6 0)
 			(hide yes)
@@
 			)
 		)
-		(property "Footprint" "lcsc:LED-SMD_4P-L2.2-W2.0-P1.00_WS2815C-2020-4P"
+		(property "Footprint" "lcsc:WS2815B-2020-V6"
 			(at 135.89 123.19 0)
 			(hide yes)
@@
 			)
 		)
-		(property "Footprint" "lcsc:LED-SMD_4P-L2.2-W2.0-P1.00_WS2815C-2020-4P"
+		(property "Footprint" "lcsc:WS2815B-2020-V6"
 			(at 157.48 78.74 0)
 			(hide yes)

Commit message: fix: rca footprint
Parts:
- J2: footprint lcsc:CONN-TH_RCJ-2122 -> lcsc:CONN-TH_RCJ-2123
Changed lines of the file:
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@@
 			)
 		)
-		(property "Footprint" "lcsc:CONN-TH_RCJ-2122"
+		(property "Footprint" "lcsc:CONN-TH_RCJ-2123"
 			(at 267.97 137.16 0)
 			(hide yes)
