File: kicad/nts_player/nts_player.kicad_sch (KiCad schematic)
At the start: 95 parts, among them J1 SJ1-3523N, J2 RCJ-2123, SW1 PEC11R-4120F-S0018, U1 ESP32-S3-DEV-KIT-N16R8, U2 LM66100DCKR, U3 TPS7A2033PDBVR, U4 TPS22918DBVR, U5 SN74AHCT1G125DBVR, U6 PCM5122PWR

Commit message: fix: placement and change resistor
Parts:
- R18, R19: LCSC Part C706320 -> C17710; MPN RT0805DRD07470RL -> 0805W8F4700T5E; Manufacturer YAGEO(国巨) -> UNI-ROYAL(厚声)
Changed lines of the file:
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@@
 			)
 		)
-		(property "Datasheet" "https://lcsc.com/product-detail/Chip-Resistor-Surface-Mount_YAGEO-RT0805DRD07470RL_C706320.html"
+		(property "Datasheet" "https://www.lcsc.com/datasheet/lcsc_datasheet_2206010200_UNI-ROYAL-Uniroyal-Elec-0805W8F4700T5E_C17710.pdf"
 			(at 278.13 31.75 0)
 			(hide yes)
@@
 			)
 		)
-		(property "Manufacturer" "YAGEO(国巨)"
+		(property "Manufacturer" "UNI-ROYAL(厚声)"
 			(at 280.67 31.75 0)
 			(hide yes)
@@
 			)
 		)
-		(property "MPN" "RT0805DRD07470RL"
+		(property "MPN" "0805W8F4700T5E"
 			(at 283.21 31.75 0)
 			(hide yes)
@@
 			)
 		)
-		(property "LCSC Part" "C706320"
+		(property "LCSC Part" "C17710"
 			(at 285.75 31.75 0)
 			(hide yes)
@@
 			)
 		)
-		(property "Datasheet" "https://lcsc.com/product-detail/Chip-Resistor-Surface-Mount_YAGEO-RT0805DRD07470RL_C706320.html"
+		(property "Datasheet" "https://www.lcsc.com/datasheet/lcsc_datasheet_2206010200_UNI-ROYAL-Uniroyal-Elec-0805W8F4700T5E_C17710.pdf"
 			(at 278.13 48.26 0)
 			(hide yes)
@@
 			)
 		)
-		(property "Manufacturer" "YAGEO(国巨)"
+		(property "Manufacturer" "UNI-ROYAL(厚声)"
 			(at 280.67 48.26 0)
 			(hide yes)
@@
 			)
 		)
-		(property "MPN" "RT0805DRD07470RL"
+		(property "MPN" "0805W8F4700T5E"
 			(at 283.21 48.26 0)
 			(hide yes)
@@
 			)
 		)
-		(property "LCSC Part" "C706320"
+		(property "LCSC Part" "C17710"
 			(at 285.75 48.26 0)
 			(hide yes)
