File: kicad/nts_player/nts_player.kicad_pcb (KiCad board)
At the start: 2 copper layers, 94 parts, among them J1 SJ1-3523N, SW1 PEC11R-4120F-S0018, U1 ESP32-S3-DEV-KIT-N16R8, U2 LM66100DCKR, U3 TPS7A2033PDBVR, U4 TPS22918DBVR, U5 SN74AHCT1G125DBVR, U6 PCM5122PWR

Commit message: fix: rca footprint
Parts:
- added J2: RCJ-2123, lcsc:CONN-TH_RCJ-2123, F.Cu at (139.0, 152.5)

Commit message: feat: work on layout
Parts:
- C1, C13, C14, C15, C19, C2, C20, C24, C25, C26, C27, C3, C31, C32, C33, C4, C40, C41, C42, C43, C44, C45, C5, C6, C7, C8, C9, D1, FB1, FB2, J1, J2, R1, R10, R11, R12, R13, R14, R15, R16, R17, R18, R19, R2, R3, R4, R5, R6, R7, R8, R9, U1, U2, U3, U4, U5, U6, USB2: moved to B.Cu
- moved C5 132.5 mm to (236.4, 54.2), turned to 180 degrees
- moved LED14 122.7 mm to (29.6, 136.2)
- moved LED13 119.5 mm to (37.6, 147.2)
- moved J2 119.3 mm to (159.8, 35.0), turned to -90 degrees
- moved LED15 118.8 mm to (30.4, 121.1)
- moved C4 118.1 mm to (236.0, 105.0), turned to 90 degrees
- moved LED16 113.7 mm to (35.0, 111.1)
- moved LED17 109.4 mm to (40.0, 104.6)
- moved C25 108.1 mm to (70.0, 100.3), turned to 180 degrees
- moved R2 103.9 mm to (236.5, 60.5)
- moved U4 103.7 mm to (70.2, 104.1), turned to -90 degrees
- moved R14 102.4 mm to (59.2, 133.8), turned to 180 degrees
- moved C23 102.3 mm to (25.0, 121.6)
- moved LED18 101.2 mm to (49.6, 100.2)
- moved R9 100.6 mm to (236.5, 63.2), turned to 180 degrees
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Routing:
- net /OUTL: track 0.00 -> 45.7 mm, vias 0 -> 1
- net /OUTR: track 0.00 -> 41.4 mm
- net GND: track 0.00 -> 40.3 mm, vias 0 -> 33
- net VBUS: track 0.00 -> 23.1 mm
- net +3.3VDAC: track 0.00 -> 20.2 mm, vias 0 -> 5
- net /AVDD: track 0.00 -> 9.38 mm
- net Net-(U6-OUTL): track 0.00 -> 7.15 mm
- net Net-(U6-OUTR): track 0.00 -> 7.11 mm
- net Net-(U6-VNEG): track 0.00 -> 5.30 mm
- net /LDOO: track 0.00 -> 4.85 mm
- net /+5V_LDO_IN: track 0.00 -> 4.37 mm
- net /CAPP: track 0.00 -> 4.14 mm
- net /CAPM: track 0.00 -> 2.53 mm
- net +5V: track 0.00 -> 1.73 mm, vias 0 -> 2
- net Net-(USB2-CC1): track 0.00 -> 1.63 mm
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- added copper zone on In1.Cu, net +3.3VDAC
Other:
- copper layers 2 -> 4

Commit message: feat: move stuff to top
Parts:
- C1, C13, C14, C15, C19, C2, C20, C24, C25, C26, C27, C3, C31, C32, C33, C4, C40, C41, C42, C43, C44, C45, C5, C6, C7, C8, C9, D1, FB1, FB2, R1, R10, R11, R12, R13, R14, R15, R16, R17, R18, R19, R2, R3, R4, R5, R6, R7, R8, R9, U2, U3, U4, U5, U6: moved to F.Cu
- moved C3 89.3 mm to (140.1, 71.2)
- moved R14 89.3 mm to (136.8, 89.5)
- moved SW1 89.3 mm to (140.0, 80.2)
- moved C2 89.3 mm to (136.0, 91.8)
- moved R8 89.3 mm to (142.5, 91.8)
- moved R7 89.2 mm to (137.6, 91.7)
- moved C1 89.1 mm to (144.1, 91.8)
- moved R15 89.1 mm to (143.2, 89.5)
- moved R13 85.9 mm to (106.1, 41.8)
- moved C9 84.4 mm to (140.5, 68.5), turned to 0 degrees
- moved USB2 83.3 mm to (107.4, 34.5)
- moved C6 82.2 mm to (109.2, 45.9), turned to 0 degrees
- moved C10 82.0 mm to (140.5, 59.0), turned to 180 degrees
- moved LED1 81.8 mm to (140.0, 62.0)
- moved C11 81.6 mm to (175.3, 101.2)
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Routing:
- net Net-(USB2-CC2): track 1.62 -> 6.91 mm, vias 0 -> 1
- net /OUTR: track 41.4 -> 46.6 mm
- net Net-(USB2-CC1): track 1.63 -> 5.88 mm, vias 0 -> 1
- net /OUTL: track 45.7 -> 48.9 mm, vias 1 -> 0
- net VBUS: track 23.1 -> 26.0 mm, vias 0 -> 2
- net GND: vias 33 -> 49
- added copper zone on F.Cu, net GND
Other:
- board outline added: 100 x 100 mm

Commit message: feat: arrange LEDs
Parts:
- removed the C39 at (119.8, 65.2)
- removed the LED18 at (124.1, 66.8)
- added C10: 0.1uF, lcsc:C0603, F.Cu at (140.0, 62.0)
- added LED1: WS2812B-2020-V6, lcsc:WS2815B-2020-V6, F.Cu at (140.0, 60.0)
- moved C12 31.6 mm to (124.4, 89.0), turned to 120 degrees
- moved C18 30.1 mm to (122.3, 83.1), turned to 100 degrees
- moved C38 29.1 mm to (128.4, 93.8), turned to 140 degrees
- moved C35 28.8 mm to (133.8, 96.9), turned to 160 degrees
- moved C29 28.2 mm to (140.0, 98.0), turned to 180 degrees
- moved C22 27.3 mm to (146.2, 96.9), turned to -160 degrees
- moved LED13 26.1 mm to (122.7, 90.0), turned to -60 degrees
- moved C17 26.0 mm to (151.6, 93.8), turned to -140 degrees
- moved C23 25.5 mm to (122.3, 76.9), turned to 80 degrees
- moved LED14 25.2 mm to (120.3, 83.5), turned to -80 degrees
- moved LED12 23.6 mm to (127.1, 95.3), turned to -40 degrees
- moved C11 23.2 mm to (155.6, 89.0), turned to -120 degrees
- moved LED11 22.7 mm to (133.2, 98.8), turned to -20 degrees
- moved LED10 22.0 mm to (140.0, 100.0)
- moved LED9 21.8 mm to (146.8, 98.8), turned to 20 degrees
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- renumbered C10 to C39, LED1 to LED18
Connections:
- C39 pad 1: +5VL -> GND
- C39 pad 2: GND -> +5VL
- LED18 pad 1: Net-(LED1-DO) -> unconnected-(LED18-DO-Pad1)
- LED18 pad 3: /LED_D -> Net-(LED17-DO)
Routing:
- net +5VL: track 0.00 -> 48.9 mm, vias 0 -> 19
- net GND: track 40.3 -> 75.6 mm, vias 49 -> 86
