File: kicad/nts_player/nts_player.kicad_pcb (KiCad board)
At the start: 4 copper layers, 100 x 100 mm, 95 parts, among them J1 SJ1-3523N, J2 RCJ-2123, SW1 PEC11R-4120F-S0018, U1 ESP32-S3-DEV-KIT-N16R8, U2 LM66100DCKR, U3 TPS7A2033PDBVR, U4 TPS22918DBVR, U5 SN74AHCT1G125DBVR, U6 PCM5122PWR

Commit message: feat: work on pcb
Parts:
- removed C9: 100uF, lcsc:C1206
- added C46: 10uF, lcsc:C1206, F.Cu at (115.9, 79.9)
- moved C5 126.1 mm to (110.8, 55.0)
- moved C4 126.1 mm to (110.0, 105.7)
- moved R1 126.1 mm to (110.7, 81.8)
- moved R10 126.1 mm to (110.7, 66.5)
- moved R11 126.1 mm to (110.7, 69.0)
- moved R2 126.1 mm to (110.7, 61.3)
- moved R3 126.1 mm to (110.7, 89.3)
- moved R4 126.1 mm to (110.7, 102.0)
- moved R5 126.1 mm to (110.7, 96.8)
- moved R6 126.1 mm to (110.7, 99.5)
- moved R9 126.1 mm to (110.7, 64.0)
- moved U1 126.1 mm to (95.8, 80.3)
- moved C25 26.0 mm to (125.9, 81.3)
- moved C13 25.6 mm to (118.3, 79.9), turned to -90 degrees
- moved U4 24.1 mm to (121.8, 80.0), turned to 180 degrees
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- renumbered LED10 to LED1
Connections:
- LED1 pad 1: Net-(LED10-DO) -> Net-(LED1-DO)
- LED1 pad 3: Net-(LED10-DI) -> /LED_D
Routing:
- net GND: track 75.6 -> 93.5 mm, vias 86 -> 95
- net +5V: track 1.73 -> 11.3 mm, vias 2 -> 3
- net +5VL: track 48.9 -> 57.3 mm, vias 19 -> 21
- net +3V3: track 0.00 -> 6.75 mm
- net /CLICK: track 0.00 -> 5.36 mm
- net Net-(U5-Y): track 0.00 -> 3.08 mm
- net /LED_D: track 0.00 -> 3.01 mm
- net Net-(U1-GPIO5): track 0.00 -> 2.83 mm
- net /SDA: track 0.00 -> 2.82 mm
- net Net-(U1-GPIO6): track 0.00 -> 2.81 mm
- net /LED_EN: track 0.00 -> 2.80 mm
- net Net-(U1-GPIO7): track 0.00 -> 2.80 mm
- net /DAC_EN: track 0.00 -> 2.79 mm
- net /SCL: track 0.00 -> 2.77 mm
- net /XSMT: track 0.00 -> 2.76 mm
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- added copper zone on In1.Cu, net +3V3
- added copper zone on In2.Cu, net GND
Other:
- board size 100 x 100 mm -> 120 x 100 mm

Commit message: feat: finalize pcb
Parts:
- moved C40 7.49 mm to (124.3, 77.6), turned to -90 degrees
- renumbered LED1 to LED10
Connections:
- LED10 pad 1: Net-(LED1-DO) -> Net-(LED10-DO)
- LED10 pad 3: /LED_D -> Net-(LED10-DI)
Routing:
- net /SCL: track 2.77 -> 81.9 mm, vias 0 -> 2
- net /SDA: track 2.82 -> 75.4 mm, vias 0 -> 2
- net /DAC_EN: track 2.79 -> 69.4 mm
- net /XSMT: track 2.76 -> 64.8 mm, vias 0 -> 2
- net /LRCK: track 0.00 -> 58.5 mm, vias 0 -> 2
- net /DIN: track 0.00 -> 56.8 mm, vias 0 -> 2
- net /BCK: track 0.00 -> 56.0 mm, vias 0 -> 2
- net /CLICK: track 5.36 -> 46.9 mm, vias 0 -> 2
- net +3V3: track 6.75 -> 44.4 mm, vias 0 -> 5
- net /LED_EN: track 2.80 -> 25.8 mm, vias 0 -> 2
- net GND: track 93.5 -> 97.6 mm, vias 95 -> 99
- added copper zone on In1.Cu, net +5V

Commit message: feat: finish pcb
Parts:
- added REF**: MountingHole_3.2mm_M3_Pad, MountingHole:MountingHole_3.2mm_M3_Pad, F.Cu at (195.0, 125.0)
- added REF**: MountingHole_3.2mm_M3_Pad, MountingHole:MountingHole_3.2mm_M3_Pad, F.Cu at (85.0, 125.0)
- added REF**: MountingHole_3.2mm_M3_Pad, MountingHole:MountingHole_3.2mm_M3_Pad, F.Cu at (85.0, 35.0)
- added REF**: MountingHole_3.2mm_M3_Pad, MountingHole:MountingHole_3.2mm_M3_Pad, F.Cu at (195.0, 35.0)
Routing:
- net /DATA_3V3: track 0.00 -> 63.5 mm, vias 0 -> 1
- net GND: track 97.6 -> 154.6 mm, vias 99 -> 102
- net Net-(U1-GPIO11): track 0.00 -> 43.6 mm, vias 0 -> 2
- net Net-(U1-GPIO10): track 0.00 -> 31.4 mm, vias 0 -> 2
- net Net-(LED14-DO): track 0.00 -> 6.81 mm
- net Net-(LED12-DO): track 0.00 -> 6.14 mm, vias 0 -> 2
- net Net-(LED10-DI): track 0.00 -> 5.69 mm
- net Net-(LED2-DO): track 0.00 -> 5.67 mm
- net Net-(LED11-DO): track 0.00 -> 5.67 mm
- net Net-(LED7-DO): track 0.00 -> 5.66 mm
- net Net-(LED16-DO): track 0.00 -> 5.66 mm
- net Net-(LED4-DO): track 0.00 -> 5.61 mm
- net Net-(LED13-DO): track 0.00 -> 5.61 mm
- net Net-(LED5-DO): track 0.00 -> 5.59 mm
- net Net-(LED6-DO): track 0.00 -> 5.51 mm
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
Commit message: fix: small things
Parts:
- moved C26 0.60 mm to (127.9, 78.3)
- turned C11 to 60 degrees
- turned C12 to -60 degrees
- turned C16 to 160 degrees
- turned C17 to 40 degrees
- turned C18 to -80 degrees
- turned C21 to 140 degrees
- turned C22 to 20 degrees
- turned C23 to -100 degrees
- turned C28 to 120 degrees
- turned C29 to 0 degrees
- turned C30 to -120 degrees
- turned C34 to 100 degrees
- turned C35 to -20 degrees
- turned C36 to -140 degrees
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Routing:
- net +5VL: track 57.3 -> 57.9 mm
- net GND: track 154.6 -> 154.1 mm

Commit message: fix: pour and stitching vias
Connections:
- U2 pad 3: GND -> +5V
Routing:
- net +5V: track 11.3 -> 15.7 mm, vias 3 -> 4
- net GND: track 154.1 -> 153.0 mm, vias 102 -> 307
- net /BCK: vias 2 -> 3
- added copper zone on In2.Cu, net +3.3VDAC
- added copper zone on In2.Cu, net +3V3
- added copper zone on In2.Cu, net +5V
- added copper zone on In2.Cu, net +5VL
- added copper zone on B.Cu, net GND
- added copper zone on In1.Cu, net GND
- removed copper zone on In1.Cu, net +3.3VDAC
- removed copper zone on In1.Cu, net +3V3
- removed copper zone on In1.Cu, net +5V
- removed copper zone on In1.Cu, net +5VL

Commit message: feat: various
Parts:
- removed REF**: MountingHole_3.2mm_M3_Pad, MountingHole:MountingHole_3.2mm_M3_Pad
- added H1: MountingHole_3.2mm_M3, MountingHole:MountingHole_3.2mm_M3, F.Cu at (85.0, 35.0)
- renumbered REF** to H2, REF** to H3, REF** to H4
Routing:
- net GND: vias 307 -> 306
- net /BCK: vias 3 -> 2
Changed lines of the file:
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@@
 		)
 	)
+	(footprint "MountingHole:MountingHole_3.2mm_M3"
+		(layer "F.Cu")
+		(at 85 35)
+		(property "Reference" "H1"
+			(at 0 -4.15 0)
+			(unlocked yes)
+			(layer "F.SilkS")
+			(hide yes)
+			(effects
+				(font
+					(size 1 1)
+					(line_spacing 0)
+				)
+			)
+		)
+		(property "Value" "MountingHole_3.2mm_M3"
+			(at 0 4.15 0)
+			(unlocked yes)
+			(layer "F.SilkS")
+			(hide yes)
+			(effects
+				(font
+					(size 1 1)
+					(line_spacing 0)
+				)
+			)
+		)
+		(property "Datasheet" ""
+			(at 0 0 0)
+			(layer "F.Fab")
+			(hide yes)
+			(effects
+				(font
+					(size 1.27 1.27)
+				)
+			)
+		)
+		(property "Description" ""
+			(at 0 0 0)
+			(layer "F.Fab")
+			(hide yes)
+			(effects
+				(font
+					(size 1.27 1.27)
+				)
+			)
+		)
+		(attr board_only)
+		(duplicate_pad_numbers_are_jumpers no)
+		(fp_circle
+			(center 0 0)
+			(end 3.2 0)
+			(stroke
+				(width 0.15)
+				(type default)
+			)
+			(fill no)
+			(layer "Cmts.User")
+		)
+		(fp_circle
+			(center 0 0)
+			(end 3.45 0)
+			(stroke
+				(width 0.05)
+				(type default)
+			)
+			(fill no)
+			(layer "F.CrtYd")
+		)
+		(fp_text user "${REFERENCE}"
+			(at 0 0 0)
+			(unlocked yes)
+			(layer "F.Fab")
+			(effects
+				(font
+					(size 1 1)
+					(thickness 0.15)
+				)
+			)
+		)
+		(pad "" np_thru_hole circle
+			(at 0 0)
+			(size 3.2 3.2)
+			(drill 3.2)
+			(layers "*.Cu" "*.Mask")
+		)
+		(embedded_fonts no)
+	)
 	(footprint "lcsc:C1206"
 		(layer "F.Cu")
@@
 		(descr "Mounting Hole 3.2mm, M3, generated by kicad-footprint-generator mountinghole.py")
 		(tags "mountinghole M3")
-		(property "Reference" "REF**"
+		(property "Reference" "H3"
 			(at 0 -4.15 0)
 			(layer "F.SilkS")
@@
 			)
 		)
-		(attr exclude_from_pos_files exclude_from_bom)
+		(attr board_only exclude_from_pos_files exclude_from_bom)
 		(duplicate_pad_numbers_are_jumpers no)
 		(fp_circle
@@
 		(descr "Mounting Hole 3.2mm, M3, generated by kicad-footprint-generator mountinghole.py")
 		(tags "mountinghole M3")
-		(property "Reference" "REF**"
+		(property "Reference" "H4"
 			(at 0 -4.15 0)
 			(layer "F.SilkS")
@@
 			)
 		)
-		(attr exclude_from_pos_files exclude_from_bom)
+		(attr board_only exclude_from_pos_files exclude_from_bom)
 		(duplicate_pad_numbers_are_jumpers no)
 		(fp_circle
@@
 		)
 	)
-	(footprint "MountingHole:MountingHole_3.2mm_M3_Pad"
-		(layer "F.Cu")
-		(at 85 35)
-		(descr "Mounting Hole 3.2mm, M3, generated by kicad-footprint-generator mountinghole.py")
-		(tags "mountinghole M3")
-		(property "Reference" "REF**"
-			(at 0 -4.15 0)
-			(layer "F.SilkS")
-			(hide yes)
-			(effects
-				(font
-					(size 1 1)
-					(thickness 0.15)
-				)
-			)
-		)
-		(property "Value" "MountingHole_3.2mm_M3_Pad"
-			(at 0 4.15 0)
-			(layer "F.Fab")
-			(effects
-				(font
-					(size 1 1)
-					(thickness 0.15)
-				)
-			)
-		)
-		(property "Datasheet" ""
-			(at 0 0 0)
-			(layer "F.Fab")
-			(hide yes)
-			(effects
-				(font
-					(size 1.27 1.27)
-				)
-			)
-		)
-		(property "Description" ""
-			(at 0 0 0)
-			(layer "F.Fab")
-			(hide yes)
-			(effects
-				(font
-					(size 1.27 1.27)
-				)
-			)
-		)
-		(property "KiLib_Generator" "mounting_hardware/mounting_hole"
-			(at 0 0 0)
-			(layer "F.SilkS")
-			(hide yes)
-			(effects
-				(font
-					(size 1 1)
-					(thickness 0.15)
-				)
-			)
-		)
-		(attr exclude_from_pos_files exclude_from_bom)
-		(duplicate_pad_numbers_are_jumpers no)
-		(fp_circle
-			(center 0 0)
-			(end 3.2 0)
-			(stroke
-				(width 0.15)
-				(type solid)
-			)
-			(fill no)
-			(layer "Cmts.User")
-		)
-		(fp_circle
-			(center 0 0)
-			(end 3.45 0)
-			(stroke
-				(width 0.05)
-				(type solid)
-			)
-			(fill no)
-			(layer "F.CrtYd")
-		)
-		(fp_text user "${REFERENCE}"
-			(at 0 0 0)
-			(layer "F.Fab")
-			(effects
-				(font
-					(size 1 1)
-					(thickness 0.15)
-				)
-			)
-		)
-		(pad "1" thru_hole circle
-			(at 0 0)
-			(size 6.4 6.4)
-			(drill 3.2)
-			(layers "*.Cu" "*.Mask")
-			(remove_unused_layers no)
-			(zone_connect 2)
-		)
-		(embedded_fonts no)
-	)
 	(footprint "lcsc:C0603"
 		(layer "F.Cu")
@@
 		(descr "Mounting Hole 3.2mm, M3, generated by kicad-footprint-generator mountinghole.py")
 		(tags "mountinghole M3")
-		(property "Reference" "REF**"
+		(property "Reference" "H2"
 			(at 0 -4.15 0)
 			(layer "F.SilkS")
@@
 			)
 		)
-		(attr exclude_from_pos_files exclude_from_bom)
+		(attr board_only exclude_from_pos_files exclude_from_bom)
 		(duplicate_pad_numbers_are_jumpers no)
 		(fp_circle
@@
 		(sheetname "/")
 		(sheetfile "nts_player.kicad_sch")
-		(units
-			(unit
-				(name "A")
-				(pins "3" "4" "2" "1")
-			)
-		)
 		(attr smd)
 		(duplicate_pad_numbers_are_jumpers no)
@@
 	)
 	(via
-		(at 162.45 64.9)
-		(size 0.6)
-		(drill 0.3)
-		(layers "F.Cu" "B.Cu")
-		(net "GND")
-	)
-	(via
 		(at 134.890427 63.76871)
 		(size 0.6)
@@
 		(net "/BCK")
 	)
-	(via
-		(at 160.5 64.5)
-		(size 0.6)
-		(drill 0.3)
-		(layers "F.Cu" "B.Cu")
-		(net "/BCK")
-	)

Commit message: fix: various
Parts:
- moved C40 13.9 mm to (132.6, 66.5), turned to 90 degrees
Routing:
- net GND: track 153.0 -> 155.2 mm
- net +5VL: track 57.9 -> 59.8 mm
Changed lines of the file:
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@@
 		(descr "100nF (104) ±10% 50V")
 		(property "Reference" "C39"
-			(at 2.677783 -1.381953 20)
+			(at 2.985083 -0.471972 20)
 			(layer "F.SilkS")
 			(effects
@@
 		(at 135.4 67.1 -90)
 		(property "Reference" "U5"
-			(at 0 2.2 90)
+			(at 0.05 -2.4 90)
 			(layer "F.SilkS")
 			(effects
@@
 			)
 		)
+		(property "LCSC Part" "C2862740"
+			(at 0 0 0)
+			(unlocked yes)
+			(layer "F.Fab")
+			(hide yes)
+			(effects
+				(font
+					(size 1 1)
+					(thickness 0.15)
+				)
+			)
+		)
+		(property "MPN" "TPS7A2033PDBVR"
+			(at 0 0 0)
+			(unlocked yes)
+			(layer "F.Fab")
+			(hide yes)
+			(effects
+				(font
+					(size 1 1)
+					(thickness 0.15)
+				)
+			)
+		)
+		(property "Manufacturer" "TI(德州仪器)"
+			(at 0 0 0)
+			(unlocked yes)
+			(layer "F.Fab")
+			(hide yes)
+			(effects
+				(font
+					(size 1 1)
+					(thickness 0.15)
+				)
+			)
+		)
 		(property ki_fp_filters "*SOT?23*")
 		(sheetname "/")
@@
 	(footprint "lcsc:C0603"
 		(layer "F.Cu")
-		(at 124.3 77.6 -90)
+		(at 132.6 66.5 90)
 		(descr "100nF (104) ±10% 50V")
 		(property "Reference" "C40"
-			(at -2.1 -2 180)
+			(at -2.25 -0.25 0)
 			(layer "F.SilkS")
 			(effects
@@
 		)
 		(property "Value" "0.1uF"
-			(at 0 4 90)
+			(at 0 4 -90)
 			(layer "F.Fab")
 			(effects
@@
 		)
 		(property "Datasheet" "https://lcsc.com/product-detail/Multilayer-Ceramic-Capacitors-MLCC-SMD-SMT_100nF-104-10-50V_C14663.html"
-			(at 0 0 90)
+			(at 0 0 -90)
 			(layer "F.Fab")
 			(hide yes)
@@
 		)
 		(property "Description" "100nF (104) ±10% 50V"
-			(at 0 0 90)
+			(at 0 0 -90)
 			(layer "F.Fab")
 			(hide yes)
@@
 		)
 		(property "LCSC Part" "C14663"
-			(at 0 0 90)
+			(at 0 0 -90)
 			(layer "F.Fab")
 			(hide yes)
@@
 		)
 		(property "Manufacturer" "YAGEO(国巨)"
-			(at 0 0 270)
+			(at 0 0 90)
 			(unlocked yes)
 			(layer "F.Fab")
@@
 		)
 		(property "MPN" "CC0603KRX7R9BB104"
-			(at 0 0 270)
+			(at 0 0 90)
 			(unlocked yes)
 			(layer "F.Fab")
@@
 		(duplicate_pad_numbers_are_jumpers no)
 		(fp_line
-			(start -0.28 0.71)
-			(end -1.08 0.71)
+			(start 0.28 -0.71)
+			(end 1.08 -0.71)
 			(stroke
 				(width 0.25)
@@
 		)
 		(fp_line
-			(start 0.28 0.71)
-			(end 1.08 0.71)
+			(start -0.28 -0.71)
+			(end -1.08 -0.71)
 			(stroke
 				(width 0.25)
@@
 		)
 		(fp_line
-			(start -1.39 0.4)
-			(end -1.39 -0.4)
+			(start 1.39 -0.4)
+			(end 1.39 0.4)
 			(stroke
 				(width 0.25)
@@
 		)
 		(fp_line
-			(start 1.39 -0.4)
-			(end 1.39 0.4)
+			(start -1.39 0.4)
+			(end -1.39 -0.4)
 			(stroke
 				(width 0.25)
@@
 		)
 		(fp_line
-			(start -0.28 -0.71)
-			(end -1.08 -0.71)
+			(start 0.28 0.71)
+			(end 1.08 0.71)
 			(stroke
 				(width 0.25)
@@
 		)
 		(fp_line
-			(start 0.28 -0.71)
-			(end 1.08 -0.71)
+			(start -0.28 0.71)
+			(end -1.08 0.71)
 			(stroke
 				(width 0.25)
@@
 		)
 		(fp_arc
-			(start -1.08 0.71)
-			(mid -1.299203 0.619203)
-			(end -1.39 0.4)
+			(start 1.08 -0.71)
+			(mid 1.299203 -0.619203)
+			(end 1.39 -0.4)
 			(stroke
 				(width 0.25)
@@
 		)
 		(fp_arc
-			(start 1.39 0.4)
-			(mid 1.299203 0.619203)
-			(end 1.08 0.71)
+			(start -1.39 -0.4)
+			(mid -1.299203 -0.619203)
+			(end -1.08 -0.71)
 			(stroke
 				(width 0.25)
@@
 		)
 		(fp_arc
-			(start -1.39 -0.4)
-			(mid -1.299203 -0.619203)
-			(end -1.08 -0.71)
+			(start 1.39 0.4)
+			(mid 1.299203 0.619203)
+			(end 1.08 0.71)
 			(stroke
 				(width 0.25)
@@
 		)
 		(fp_arc
-			(start 1.08 -0.71)
-			(mid 1.299203 -0.619203)
-			(end 1.39 -0.4)
+			(start -1.08 0.71)
+			(mid -1.299203 0.619203)
+			(end -1.39 0.4)
 			(stroke
 				(width 0.25)
@@
 		)
 		(fp_line
-			(start -0.8 0.4)
-			(end -0.8 -0.4)
+			(start 0.8 -0.4)
+			(end 0.8 0.4)
 			(stroke
 				(width 0.05)
@@
 		)
 		(fp_line
-			(start 0.8 0.4)
-			(end -0.8 0.4)
+			(start -0.8 -0.4)
+			(end 0.8 -0.4)
 			(stroke
 				(width 0.05)
@@
 		)
 		(fp_line
-			(start -0.8 -0.4)
-			(end 0.8 -0.4)
+			(start 0.8 0.4)
+			(end -0.8 0.4)
 			(stroke
 				(width 0.05)
@@
 		)
 		(fp_line
-			(start 0.8 -0.4)
-			(end 0.8 0.4)
+			(start -0.8 0.4)
+			(end -0.8 -0.4)
 			(stroke
 				(width 0.05)
@@
 		)
 		(fp_text user "${REFERENCE}"
-			(at 0 0 90)
+			(at 0 0 -90)
 			(layer "F.Fab")
 			(effects
@@
 		)
 		(pad "1" smd rect
-			(at -0.7 0 270)
+			(at -0.7 0 90)
 			(size 0.8 0.9)
 			(layers "F.Cu" "F.Mask" "F.Paste")
@@
 		)
 		(pad "2" smd rect
-			(at 0.7 0 270)
+			(at 0.7 0 90)
 			(size 0.8 0.9)
 			(layers "F.Cu" "F.Mask" "F.Paste")
@@
 	)
 	(segment
-		(start 124.3 76.9)
-		(end 124.3 76)
-		(width 0.3)
-		(layer "F.Cu")
-		(net "GND")
-	)
-	(segment
 		(start 173.374 65.124)
 		(end 173.374 66.094)
@@
 	)
 	(segment
+		(start 132.6 67.2)
+		(end 132.6 68.4)
+		(width 0.3)
+		(layer "F.Cu")
+		(net "GND")
+	)
+	(segment
 		(start 154.415733 89.131218)
 		(end 154.347432 89.149519)
@@
 	)
 	(segment
+		(start 132.6 68.4)
+		(end 134.45 68.4)
+		(width 0.3)
+		(layer "F.Cu")
+		(net "GND")
+	)
+	(segment
 		(start 109.36 107.02)
 		(end 109.95 106.43)
@@
 		(width 0.3)
 		(layer "F.Cu")
+		(net "+5VL")
+	)
+	(segment
+		(start 132.6 65.8)
+		(end 134.45 65.8)
+		(width 0.3)
+		(layer "F.Cu")
