File: kicad/nts_player/nts_player.kicad_pcb (KiCad board)
At the start: 4 copper layers, 120 x 100 mm, 99 parts, among them J1 SJ1-3523N, J2 RCJ-2123, SW1 PEC11R-4120F-S0018, U1 ESP32-S3-DEV-KIT-N16R8, U2 LM66100DCKR, U3 TPS7A2033PDBVR, U4 TPS22918DBVR, U5 SN74AHCT1G125DBVR, U6 PCM5122PWR

Commit message: fix: align vias
Routing:
- net GND: vias 306 -> 303
